Commit message: [ADD] Moveit package

File: ur_5e_gripper_description/urdf/ur5e_2f_85.xacro (robot description, xacro)
@@ -6,8 +6,14 @@
         <xacro:ur5e_robot prefix="" />
         <xacro:robotiq_arg2f_85 prefix=""/>
+        <link name="tcp_link"/>
         <joint name="joint_tool" type="fixed">
             <parent link="tool0"/>
             <child link="robotiq_arg2f_base_link"/>
-            <origin xyz="0 0 0.0169" rpy="0 0 0"/>
+            <origin xyz="0 0 0.0169" rpy="0 0 1.57"/>
+        </joint>
+        <joint name="joint_tcp" type="fixed">
+            <parent link="tool0"/>
+            <child link="tcp_link"/>
+            <origin xyz="0 0 0.147" rpy="0 0 0"/>
         </joint>
     </xacro:macro>
