Commit message: [ADD] moveit_config with table and camera attach

File: ur5e_2f_85_description/urdf/ur5e_2f_85_zed_mini_camera_table.xacro (robot description, xacro)
@@ -8,5 +8,5 @@
             <parent link="robot_base_1"/>
             <child link="base_link"/>
-            <origin xyz="0.0 0.0 0.00" rpy="0 0 0.0"/>
+            <origin xyz="0.0 0.0 0.00" rpy="0 0 3.18"/>
         </joint>
     </xacro:macro>
