Commit message: [ADD] Table, camera moveit package

File: ur5e_2f_85_camera_table_moveit_config/config/gazebo_ur5e_2f_85.urdf (robot description, URDF)
Before this commit: robot ur5e_2f_85, 37 links, 36 joints
Joints:
- joint robot_base: origin xyz=0.40 0.165 0.84 rpy=0 0 0 -> xyz=0.40 0.135 0.86 rpy=0 0 0
- joint table: origin xyz=0.400 -0.477 0.727 rpy=0 0 0 -> xyz=0.400 -0.477 0.74 rpy=0 0 0

File: ur5e_2f_85_description/urdf/table_and_robot_platform.xacro (robot description, xacro)
@@ -237,10 +237,10 @@
 </joint>
 <joint name="table" type="fixed">
-  <origin xyz="0.400 -0.477 0.727" rpy="0 0 0"/>
+  <origin xyz="0.400 -0.477 0.74" rpy="0 0 0"/>
   <parent link="base_link_platform"/>
   <child link="Plane-Table_1"/>
 </joint>
 <joint name="robot_base" type="fixed">
-  <origin xyz="0.40 0.165 0.84" rpy="0 0 0"/>
+  <origin xyz="0.38 0.135 0.86" rpy="0 0 0"/>
   <parent link="base_link_platform"/>
   <child link="robot_base_1"/>

Commit message: [ADD] modified robot model

File: ur5e_2f_85_camera_table_moveit_config/config/gazebo_ur5e_2f_85.urdf (robot description, URDF)
Before this commit: robot ur5e_2f_85, 37 links, 36 joints
Links:
- removed link Plane-Table_1
- removed link table_suport_sx_back_1
- added link table_1, mass 0.1; collision mesh filename=package://ur5e_2f_85_description/meshes/robot_platform/tabl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 scale=0.001 0.001 0.001; visual mesh filename=package://ur5e_2f_85_description/meshes/robot_platform/tabl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 scale=0.001 0.001 0.001
- added link table_support_sx_back_1, mass 0.1; collision mesh filename=package://ur5e_2f_85_description/meshes/robot_platform/tabl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 scale=0.001 0.001 0.001; visual mesh filename=package://ur5e_2f_85_description/meshes/robot_platform/tabl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 scale=0.001 0.001 0.001
Joints:
- joint base_link_back_left_support: child table_suport_sx_back_1 -> table_support_sx_back_1
- joint table: child Plane-Table_1 -> table_1
- joint vertical_back_left: parent table_suport_sx_back_1 -> table_support_sx_back_1

File: ur5e_2f_85_description/urdf/table_and_robot_platform copy.xacro (robot description, xacro)
@@ -163,10 +163,10 @@
 <link name="table_1">
   <!-- <inertial>
-    <origin xyz="0.40000000000000147 -0.4769999999999962 0.7212526611221979" rpy="0 0 0"/>
-    <mass value="404.2332203814961"/>
-    <inertia ixx="33.775427" iyy="33.775427" izz="67.372203" ixy="-0.0" iyz="0.0" ixz="-0.0"/>
-  </inertial> -->
-  <visual>
-    <origin xyz="-0.400 0.477 -0.74" rpy="0 0 0"/>
+    <origin xyz="0.40000000000000385 -0.47699999999999404 0.7112526611221979" rpy="0 0 0"/>
+    <mass value="247.23322038149666"/>
+    <inertia ixx="20.623205" iyy="20.623205" izz="41.205537" ixy="-0.0" iyz="0.0" ixz="0.0"/>
+  </inertial> -->
+  <visual>
+    <origin xyz="-0.400 0.477 -0.71" rpy="0 0 0"/>
     <geometry>
       <mesh filename="package://ur5e_2f_85_description/meshes/robot_platform/table_1.stl" scale="0.001 0.001 0.001"/>
@@ -175,5 +175,5 @@
   </visual>
   <collision>
-    <origin xyz="-0.400 0.477 -0.74" rpy="0 0 0"/>
+    <origin xyz="-0.400 0.477 -0.71" rpy="0 0 0"/>
     <geometry>
       <mesh filename="package://ur5e_2f_85_description/meshes/robot_platform/table_1.stl" scale="0.001 0.001 0.001"/>
@@ -183,10 +183,10 @@
 <link name="robot_base_1">
   <!-- <inertial>
-    <origin xyz="0.4000343598428915 0.1650000000000009 0.8452146550277948" rpy="0 0 0"/>
+    <origin xyz="0.40003435984289154 0.1650000000000009 0.8252146550277948" rpy="0 0 0"/>
     <mass value="4.5478768461232075"/>
     <inertia ixx="0.019419" iyy="0.019473" izz="0.038619" ixy="0.0" iyz="0.0" ixz="-1e-06"/>
   </inertial> -->
   <visual>
-    <origin xyz="-0.40 -0.165 -0.86" rpy="0 0 0"/>
+    <origin xyz="-0.40 -0.165 -0.84" rpy="0 0 0"/>
     <geometry>
       <mesh filename="package://ur5e_2f_85_description/meshes/robot_platform/robot_base_1.stl" scale="0.001 0.001 0.001"/>
@@ -195,5 +195,5 @@
   </visual>
   <collision>
-    <origin xyz="-0.40 -0.165 -0.86" rpy="0 0 0"/>
+    <origin xyz="-0.40 -0.165 -0.84" rpy="0 0 0"/>
     <geometry>
       <mesh filename="package://ur5e_2f_85_description/meshes/robot_platform/robot_base_1.stl" scale="0.001 0.001 0.001"/>

Commit message: [ADD] baseline for AI controller

File: ur5e_2f_85_camera_table_moveit_config/config/gazebo_ur5e_2f_85.urdf (robot description, URDF)
Before this commit: robot ur5e_2f_85, 37 links, 36 joints
Joints:
- joint robot_base: origin xyz=0.40 0.135 0.86 rpy=0 0 0 -> xyz=0.38 0.135 0.86 rpy=0 0 0
